File: xiao_spread.kicad_pcb (KiCad board)
At the start: 2 copper layers, 121.5 x 92.9 mm, 48 parts, among them J1 B5B-XH-A_LF__SN_, SW1 RotaryEncoder_Switch, U2 SeeeduinoXIAO

Commit message: user update
Routing:
- net Row_3: track 62.8 -> 62.1 mm
Other:
- board text added: "Xiao face DOWN"
- board text added: "Xiao face UP"
- board text added: "凱"
